Commit message: Change joint2 to revolute, need better coverage of tests

File: moveit_planners/chomp/chomp_interface/test/rrbot.xacro (robot description, xacro)
@@ -78,5 +78,5 @@
     </inertial>
   </link>
-  <joint name="joint2" type="continuous">
+  <joint name="joint2" type="revolute">
     <parent link="link2"/>
     <child link="link3"/>
@@ -84,5 +84,5 @@
     <axis xyz="0 1 0"/>
     <dynamics damping="0.7"/>
-    <limit effort="20" velocity="${2*PI}" />
+    <limit upper="${-PI/2.0}" lower="${PI/2.0}" effort="20" velocity="${2*PI}" />
   </joint>
   <!-- Top Link -->

Commit message: [PI/2,-PI/2] is a bad interval, fix: [-PI/2, PI/2]

File: moveit_planners/chomp/chomp_interface/test/rrbot.xacro (robot description, xacro)
@@ -84,5 +84,5 @@
     <axis xyz="0 1 0"/>
     <dynamics damping="0.7"/>
-    <limit upper="${-PI/2.0}" lower="${PI/2.0}" effort="20" velocity="${2*PI}" />
+    <limit upper="${PI/2.0}" lower="${-PI/2.0}" effort="20" velocity="${2*PI}" />
   </joint>
   <!-- Top Link -->

Commit message: Add collision box to urdf

File: moveit_planners/chomp/chomp_interface/test/rrbot.xacro (robot description, xacro)
@@ -8,5 +8,4 @@
   <xacro:property name="height2" value="1" /> <!-- Link 2 -->
   <xacro:property name="height3" value="1" /> <!-- Link 3 -->
-  <xacro:property name="camera_link" value="0.05" /> <!-- Size of square 'camera' box -->
   <xacro:property name="axel_offset" value="0.05" /> <!-- Space btw top of beam and the each joint -->
   <material name="black">
@@ -110,3 +109,31 @@
     </inertial>
   </link>
+  <!-- A box to test collision checking against -->
+  <joint name="box_to_world_joint" type="fixed">
+    <parent link="world"/>
+    <child link="obstacle_box_link"/>
+    <origin xyz="1.0 0.2 2.0"/>
+  </joint>
+  <link name="obstacle_box_link">
+    <collision>
+      <origin xyz="0 0 0" rpy="0 0 0"/>
+      <geometry>
+        <box size="0.2 0.2 0.2"/>
+      </geometry>
+    </collision>
+    <visual>
+      <origin xyz="0 0 0" rpy="0 0 0"/>
+      <geometry>
+        <box size="0.2 0.2 0.2"/>
+      </geometry>
+    </visual>
+    <inertial>
+      <origin xyz="0 0 ${height3/2 - axel_offset}" rpy="0 0 0"/>
+      <mass value="1"/>
+      <inertia
+        ixx="1.0" ixy="0.0" ixz="0.0"
+        iyy="1.0" iyz="0.0"
+        izz="1.0"/>
+    </inertial>
+  </link>
 </robot>
